File: Hardware/ESS-STM-Hardware.kicad_sch (KiCad schematic)
At the start: 14 parts, among them J1 Conn_01x06_Pin, J2 Conn_01x06_Pin, J3 Conn_01x06_Pin, J4 Conn_ARM_SWD_TagConnect_TC2030, U1 STM32C011F4Ux, U2 24AA02-OT

Commit message: Finished Schematic
Parts:
- added C4, C5: 4.7u, Capacitor_SMD:C_0603_1608Metric, symbol Device:C
- added U3: AP7361C-33E, Package_TO_SOT_SMD:SOT-223-3_TabPin2, symbol Regulator_Linear:AP7361C-33E
- J1, J2, J3: footprint (none) -> Connector_JST:JST_PH_S5B-PH-SM4-TB_1x05-1MP_P2.00mm_Horizontal
Connections:
- net +3.3V_CON is gone; now on net +3.3V_Con: J2.6 (Pin_6), R4.1
- net +3.3V_MCU: now also C5.1, U3.3 (VO)
- net +5V: now also C4.1, U3.1 (VI)
- net GND: now also C4.2, C5.2, U3.2 (GND)
- no-connect marks 4 -> 13
Other:
- removed sheet Power Regulators
- note added: "Power Inputs From Console"
- note added: "STM32 Power"
- moved on the sheet: C1, C2, C3, J4, R1, R2, U2

Commit message: Some changes to board design
Parts:
- J1, J2, J3: symbol Connector:Conn_01x06_Pin -> Connector:Conn_01x05_Pin
Connections:
- net +3.3V_Con: now also J1.5 (Pin_5), J2.5 (Pin_5), J3.5 (Pin_5); no longer J1.6 (Pin_6), J2.6 (Pin_6), J3.6 (Pin_6)
- net GC_Data: now also U1.6 (PA1); no longer U1.13 (PA8)
- net N64_Data: now also U1.5 (PA0); no longer U1.12 (PA7)
- net at D1.2 (A): now also U1.10 (PA5); no longer U1.5 (PA0)
- no-connect marks 13 -> 10
Other:
- moved on the sheet: D1
