File: Hardware/ESS-STM-Hardware.kicad_pcb (KiCad board)
At the start: 2 copper layers, 55 x 40 mm, 17 parts, among them J1 Conn_01x06_Pin, J2 Conn_01x06_Pin, J3 Conn_01x06_Pin, J4 Conn_ARM_SWD_TagConnect_TC2030, U1 STM32C011F4Ux, U2 24AA02-OT, U3 AP7361C-33E

Commit message: Some changes to board design
Parts:
- added ?: , , F.Cu at (154.0, 113.0)
- added REF**: MountingHole_3.2mm_M3_ISO7380_Pad, MountingHole:MountingHole_3.2mm_M3_ISO7380_Pad, F.Cu at (154.0, 87.0)
- moved C1 110.3 mm to (137.5, 100.0), turned to 180 degrees
- moved R3 105.8 mm to (136.5, 105.0), turned to -90 degrees
- moved C2 105.4 mm to (137.5, 98.5), turned to 180 degrees
- moved R4 104.4 mm to (138.5, 93.0), turned to 180 degrees
- moved C3 104.0 mm to (138.5, 96.0)
- moved C5 103.4 mm to (139.5, 106.0)
- moved C4 100.8 mm to (142.5, 106.0), turned to 180 degrees
- moved R2 95.2 mm to (147.5, 90.5), turned to 180 degrees
- moved R1 95.1 mm to (147.5, 88.5), turned to 180 degrees
- moved D1 6.52 mm to (146.0, 103.5)
- moved U2 5.03 mm to (145.0, 95.5), turned to -90 degrees
- moved J4 4.59 mm to (141.5, 88.0)
- moved J3 3.54 mm to (153.5, 99.0)
- moved U1 1.39 mm to (141.5, 99.5)
Connections:
- J1 pad 5: unconnected-(J1-Pin_5-Pad5) -> +3.3V_Con
- J2 pad 5: unconnected-(J2-Pin_5-Pad5) -> +3.3V_Con
- J3 pad 5: unconnected-(J3-Pin_5-Pad5) -> +3.3V_Con
- U1 pad 10: unconnected-(U1-PA5-Pad10) -> Net-(D1-A)
- U1 pad 12: N64_Data -> unconnected-(U1-PA7-Pad12)
- U1 pad 13: GC_Data -> unconnected-(U1-PA8-Pad13)
- U1 pad 5: Net-(D1-A) -> N64_Data
- U1 pad 6: unconnected-(U1-PA1-Pad6) -> GC_Data
Routing:
- net +5V: track 0.00 -> 53.0 mm, vias 0 -> 3
- net +3.3V_Con: track 0.00 -> 45.1 mm, vias 0 -> 4
- net GC_Data: track 0.00 -> 23.5 mm, vias 0 -> 2
- net _RESET: track 0.00 -> 20.4 mm, vias 0 -> 2
- net SWCLK: track 0.00 -> 15.5 mm
- net N64_Data: track 0.00 -> 13.6 mm, vias 0 -> 2
- net GND: track 0.00 -> 12.9 mm, vias 0 -> 29
- net +3.3V_MCU: track 0.00 -> 12.7 mm, vias 0 -> 12
- net I2C_SDA: track 0.00 -> 12.4 mm
- net SWDIO: track 0.00 -> 11.9 mm
- net I2C_SCL: track 0.00 -> 10.6 mm
- net Console_DO: track 0.00 -> 7.88 mm
- net Net-(D1-A): track 0.00 -> 6.05 mm
- added copper zone on In2.Cu, net +3.3V_MCU
- added copper zone on B.Cu, net GND
- added copper zone on F.Cu, net GND
- added copper zone on In1.Cu, net GND
Other:
- board size 55 x 40 mm -> 33.6 x 35 mm
- copper layers 2 -> 4
- board text added: "2024-11-10"
- board text added: "Console"
- board text added: "Ess Adapter"
- board text added: "GC"
- board text added: "N64"
- board text added: "Rev 0"

Commit message: Finish PCB Rev 0 Design
Routing:
- net SWDIO: track 11.9 -> 17.7 mm, vias 0 -> 2
- net GND: vias 29 -> 31
Other:
- board text added: "2025-01-19"
- board text removed: "2024-11-10"
Changed lines of the file:
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@@
 	(title_block
 		(title "ESS-STM")
-		(date "2024-11-05")
+		(date "2025-01-19")
 		(rev "0")
 	)
@@
 			(outputformat 1)
 			(mirror no)
-			(drillshape 1)
+			(drillshape 0)
 			(scaleselection 1)
-			(outputdirectory "")
+			(outputdirectory "GerberOut/")
 		)
 	)
@@
 			(net 2 "GND")
 			(pintype "passive")
+			(zone_connect 2)
 		)
 		(model "${KICAD8_3DMODEL_DIR}/Capacitor_SMD.3dshapes/C_0603_1608Metric.wrl"
@@
 			(net 2 "GND")
 			(pintype "passive")
+			(zone_connect 2)
 		)
 		(model "${KICAD8_3DMODEL_DIR}/Capacitor_SMD.3dshapes/C_0603_1608Metric.wrl"
@@
 			(remove_unused_layers no)
 			(net 2 "GND")
+			(zone_connect 2)
 		)
 	)
@@
 			(remove_unused_layers no)
 			(net 2 "GND")
+			(zone_connect 2)
 		)
 	)
@@
 			(pinfunction "Pin_3")
 			(pintype "passive")
+			(zone_connect 2)
 		)
 		(pad "4" smd roundrect
@@
 			(pinfunction "Pin_4")
 			(pintype "passive")
+			(zone_connect 2)
 		)
 		(pad "5" smd roundrect
@@
 			(net 2 "GND")
 			(pintype "passive")
+			(zone_connect 2)
 		)
 		(model "${KICAD8_3DMODEL_DIR}/Capacitor_SMD.3dshapes/C_0603_1608Metric.wrl"
@@
 			(pinfunction "WP")
 			(pintype "input")
+			(zone_connect 2)
 		)
 		(model "${KICAD8_3DMODEL_DIR}/Package_TO_SOT_SMD.3dshapes/SOT-23-5.wrl"
@@
 			(pinfunction "Pin_3")
 			(pintype "passive")
+			(zone_connect 2)
 		)
 		(pad "4" smd roundrect
@@
 			(pinfunction "Pin_4")
 			(pintype "passive")
+			(zone_connect 2)
 		)
 		(pad "5" smd roundrect
@@
 			(pinfunction "K")
 			(pintype "passive")
+			(zone_connect 2)
 		)
 		(pad "2" smd roundrect
@@
 			(net 2 "GND")
 			(pintype "passive")
+			(zone_connect 2)
 		)
 		(model "${KICAD8_3DMODEL_DIR}/Capacitor_SMD.3dshapes/C_0603_1608Metric.wrl"
@@
 			(net 2 "GND")
 			(pintype "passive")
+			(zone_connect 2)
 		)
 		(model "${KICAD8_3DMODEL_DIR}/Diode_SMD.3dshapes/D_0603_1608Metric.wrl"
@@
 			(pinfunction "GND")
 			(pintype "power_in")
+			(zone_connect 2)
 		)
 		(pad "2" smd roundrect
@@
 			(pinfunction "GND")
 			(pintype "power_in")
+			(zone_connect 2)
 		)
 		(pad "3" smd roundrect
@@
 			(pinfunction "Pin_3")
 			(pintype "passive")
+			(zone_connect 2)
 		)
 		(pad "4" smd roundrect
@@
 			(pinfunction "Pin_4")
 			(pintype "passive")
+			(zone_connect 2)
 		)
 		(pad "5" smd roundrect
@@
 	)
 	(gr_rect
-		(start 130.7 90.8)
-		(end 134.9 94.2)
-		(stroke
-			(width 0.2)
-			(type solid)
-		)
-		(fill solid)
-		(layer "F.Cu")
-		(net 2)
-	)
-	(gr_rect
-		(start 144 102.4)
-		(end 145.452542 105.4)
-		(stroke
-			(width 0.2)
-			(type solid)
-		)
-		(fill solid)
-		(layer "F.Cu")
-		(net 2)
-	)
-	(gr_rect
-		(start 148.8 96.5)
-		(end 154.8 99.5)
-		(stroke
-			(width 0.2)
-			(type solid)
-		)
-		(fill solid)
-		(layer "F.Cu")
-		(net 2)
-	)
-	(gr_rect
-		(start 140.4 105.4)
-		(end 142 114)
-		(stroke
-			(width 0.2)
-			(type solid)
-		)
-		(fill solid)
-		(layer "F.Cu")
-		(net 2)
-	)
-	(gr_rect
-		(start 129.6 108.101012)
-		(end 134.8 111)
-		(stroke
-			(width 0.2)
-			(type solid)
-		)
-		(fill solid)
-		(layer "F.Cu")
-		(net 2)
-	)
-	(gr_rect
 		(start 137.2 107.4)
 		(end 139.8 111.2)
@@
 		(net 1)
 	)
-	(gr_rect
-		(start 140.4 110.6)
-		(end 144.6 113)
-		(stroke
-			(width 0.2)
-			(type solid)
-		)
-		(fill solid)
-		(layer "F.Cu")
-		(net 2)
-	)
-	(gr_rect
-		(start 136 97.8)
-		(end 137.2 102)
-		(stroke
-			(width 0.2)
-			(type solid)
-		)
-		(fill solid)
-		(layer "F.Cu")
-		(net 2)
-	)
-	(gr_rect
-		(start 138.2 112.6)
-		(end 143.8 115.8)
-		(stroke
-			(width 0.2)
-			(type solid)
-		)
-		(fill solid)
-		(layer "F.Cu")
-		(net 2)
-	)
 	(gr_line
 		(start 156.616087 117.5)
@@
 		)
 	)
-	(gr_text "2024-11-10"
+	(gr_text "2025-01-19"
 		(at 144 116 0)
 		(layer "B.SilkS")
@@
 	)
 	(via
+		(at 135.2 93)
+		(size 0.6)
+		(drill 0.3)
+		(layers "F.Cu" "B.Cu")
+		(net 2)
+	)
+	(via
 		(at 144.2 104.8)
 		(size 0.6)
@@
 		(net 2)
 	)
+	(via
+		(at 135.2 92)
+		(size 0.6)
+		(drill 0.3)
+		(layers "F.Cu" "B.Cu")
+		(net 2)
+	)
 	(segment
 		(start 139 90.8)
@@
 	)
 	(segment
-		(start 141.4437 94.4437)
-		(end 142 95)
-		(width 0.15)
+		(start 142.4 86.465)
+		(end 142.4 84)
+		(width 0.2)
 		(layer "F.Cu")
 		(net 10)
 	)
 	(segment
-		(start 142 95)
-		(end 142 98.2)
-		(width 0.15)
+		(start 141.975 95.6)
+		(end 142 95.625)
+		(width 0.2)
 		(layer "F.Cu")
 		(net 10)
@@
 	(segment
 		(start 142.095 86.77)
-		(end 141.4437 87.4213)
-		(width 0.15)
+		(end 142.4 86.465)
+		(width 0.2)
 		(layer "F.Cu")
 		(net 10)
 	)
 	(segment
-		(start 141.4437 87.4213)
-		(end 141.4437 94.4437)
-		(width 0.15)
+		(start 142 95.625)
+		(end 142 98.2)
+		(width 0.2)
 		(layer "F.Cu")
 		(net 10)
 	)
+	(via
+		(at 141.975 95.6)
+		(size 0.6)
+		(drill 0.3)
+		(layers "F.Cu" "B.Cu")
+		(net 10)
+	)
+	(via
+		(at 142.4 84)
+		(size 0.6)
+		(drill 0.3)
+		(layers "F.Cu" "B.Cu")
+		(net 10)
+	)
+	(segment
+		(start 142.4 87.6)
+		(end 141.6 88.4)
+		(width 0.2)
+		(layer "B.Cu")
+		(net 10)
+	)
+	(segment
+		(start 141.4687 95.0937)
+		(end 141.975 95.6)
+		(width 0.2)
+		(layer "B.Cu")
+		(net 10)
+	)
+	(segment
+		(start 141.4687 93.2)
+		(end 141.4687 95.0937)
+		(width 0.2)
+		(layer "B.Cu")
+		(net 10)
+	)
+	(segment
+		(start 141.4687 88.5313)
+		(end 141.4687 93.2)
+		(width 0.2)
+		(layer "B.Cu")
+		(net 10)
+	)
+	(segment
+		(start 141.6 88.4)
+		(end 141.4687 88.5313)
+		(width 0.2)
+		(layer "B.Cu")
+		(net 10)
+	)
+	(segment
+		(start 142.4 84)
+		(end 142.4 87.6)
+		(width 0.2)
+		(layer "B.Cu")
+		(net 10)
+	)
